Commit message: Add AMCL watchdog, goal checker guard and controller recovery
Fleet manager now uses the four-condition priority order, ignores plans of
robots with no active goal, and restarts a controller_server whose local
costmap stops updating, then resends the goal. New amcl_watchdog_node
re-seeds AMCL when its pose goes stale. New GuardedGoalChecker plugin
rejects the default-constructed goal pose that Nav2 passes after a failed
map->odom lookup.

Comments removed from all source files and the README rewritten.

File: src/amr_description/urdf/amr_gazebo.xacro (robot description, xacro)
@@ -40,8 +40,3 @@
         </plugin>
     </gazebo>
-    <!-- gz-sim-sensors-system is NOT declared here: it owns the shared
-         rendering scene, so it must be loaded exactly once per world (see
-         world/maze.sdf), not once per spawned robot model. Two copies (e.g.
-         one per robot in a multi-robot bringup) crash with "Scene already
-         exists with name: scene". -->
 </robot>

File: src/amr_description/urdf/camera.xacro (robot description, xacro)
@@ -23,5 +23,4 @@
     </link>
     <link name="camera_link_optical" />
-    <!-- CAMERA JOINT -->
     <joint name="camera_joint" type="fixed">
         <parent link="amr_body" />
@@ -29,5 +28,4 @@
         <origin xyz="0.21 -0.04 0.195" rpy="0 0 0" />
     </joint>
-    <!-- OPTICAL FRAME JOINT -->
     <joint name="camera_optical_joint" type="fixed">
         <parent link="camera_link" />

File: src/amr_description/urdf/depth_camera.xacro (robot description, xacro)
@@ -23,5 +23,4 @@
     </link>
     <link name="depth_camera_link_optical" />
-    <!-- CAMERA JOINT -->
     <joint name="depth_camera_joint" type="fixed">
         <parent link="amr_body" />
@@ -29,10 +28,8 @@
         <origin xyz="0.21 -0.04 0.195" rpy="0 0 0" />
     </joint>
-    <!-- OPTICAL FRAME JOINT -->
     <joint name="depth_camera_optical_joint" type="fixed">
         <parent link="depth_camera_link" />
         <child link="depth_camera_link_optical" />
         <origin xyz="0 0 0" rpy="-1.57 0 -1.57"  />
-        <!-- <origin xyz="0 0 0" rpy="-1.57 0 -1.57" /> -->
     </joint>
     <gazebo reference="depth_camera_link">
@@ -49,14 +46,6 @@
                     <far>10</far>
                 </clip>
-                <!--
-                <noise>
-                    <type>gaussian</type>
-                    <mean>0.0</mean>
-                    <stddev>0.007</stddev>
-                </noise>
-                -->
                 <optical_frame_id>depth_camera_link_optical</optical_frame_id>
                 <camera_info_topic>depth_camera_link_optical</camera_info_topic>
-               <!-- <camera_info_topic>camera/camera_info</camera_info_topic> -->
             </camera>
             <always_on>1</always_on>
@@ -64,5 +53,4 @@
             <visualize>true</visualize>
             <topic>/depth_camera/depth/image_raw</topic>
-            <!-- <gz_frame_id>depth_camera_link_optical</gz_frame_id> -->
         </sensor>
     </gazebo>

File: src/amr_description/urdf/lidar.xacro (robot description, xacro)
@@ -9,9 +9,7 @@
       <material name="transparent" />
     </visual>
-    <!--Inertial Tag-->
     <xacro:box_inertia m="0.16" l="0.06" w="0.06" h="0.08"
                         xyz="0 0 0" rpy="0 0 0" />
   </link>
-  <!-- ===== JOINT: attach to amr_body ===== -->
   <joint name="${prefix_}lidar_joint" type="fixed">
     <parent link="${prefix_}amr_body"/>

File: src/amr_description/urdf/properties.xacro (robot description, xacro)
@@ -2,20 +2,18 @@
 <robot xmlns:xacro="http://www.ros.org/wiki/xacro">
     <material name="amr_body_color">
-        <color rgba="0.00 0.65 0.58 1.0"/> <!-- Teal -->
+        <color rgba="0.00 0.65 0.58 1.0"/>
     </material>
     <material name="amr_wheel_color">
-        <color rgba="0.18 0.24 0.27 1.0"/> <!-- Charcoal -->
+        <color rgba="0.18 0.24 0.27 1.0"/>
     </material>
     <material name="amr_lift_color">
-        <color rgba="1.00 0.54 0.25 1.0"/> <!-- Orange -->
+        <color rgba="1.00 0.54 0.25 1.0"/>
     </material>
     <material name="amr_caster_color">
-        <color rgba="0.00 0.46 0.71 1.0"/> <!-- Electric Blue Caster Wheel-->
+        <color rgba="0.00 0.46 0.71 1.0"/>
     </material>
     <material name="transparent">
-        <color rgba="0.00 0.65 0.58 0.1"/> <!-- Teal -->
+        <color rgba="0.00 0.65 0.58 0.1"/>
     </material>
-                    <!-- INTERIA XACRO MACRO -->
-    <!-- BODY INTERIA -->
     <xacro:macro name="box_inertia" params="m l w h xyz rpy" >
         <inertial>
@@ -27,5 +25,4 @@
         </inertial>
     </xacro:macro>
-    <!-- WHEEL INTERIA -->
     <xacro:macro name="cylinder_inertia" params="m r h xyz rpy" >
         <inertial>
@@ -37,5 +34,4 @@
         </inertial>
     </xacro:macro>
-    <!-- CASTER WHEEL MACRO -->
     <xacro:macro name="sphere_inertia" params="m r o_xyz o_rpy">
         <inertial>

File: src/amr_description/urdf/stand.xacro (robot description, xacro)
@@ -9,5 +9,4 @@
             </geometry>
         </visual>
-        <!--COLLISION TAG-->
         <collision>
             <origin xyz="0.0 0.0 -0.24" rpy="0.0 0.0 0.0"/>
@@ -17,9 +16,7 @@
             </geometry>
         </collision>
-        <!--Inertial Tag-->
         <xacro:box_inertia m="240.0" l="1.250" w="0.9" h="0.26"
                             xyz="0.0 0.0 0.13" rpy="0.0 0.0 0.0" />
     </link>
-    <!-- CAMERA JOINT -->
     <joint name="${prefix_}stand_joint" type="fixed">
         <parent link="${prefix_}base_link" />
